File: SX1255-STM32H723 HAT.kicad_pcb (KiCad board)
At the start: 2 copper layers, 36 parts, among them IC1 SX1255, J1 TX_SMA, J2 RX_SMA, J3 STM-L, J4 STM-R, U1 MCP1703Ax-330xxMB, X1 TA0692A, Y1 32MHz

Commit message: Add files via upload
Parts:
- D1: value PWR-LED Orange -> PWR
- J1: value TX_SMA -> TX_ANT
- J2: value RX_SMA -> RX_ANT
- moved REF** 0.50 mm to (174.2, 86.5)
Other:
- board outline added: 77 x 44.2 mm
Changed lines of the file:
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@@
 		(tags "Through hole socket strip THT 2x30 2.54mm double row")
 		(property "Reference" "J4"
-			(at -1.27 -2.77 90)
+			(at -5.54 0.14 90)
 			(layer "F.SilkS")
 			(effects
@@
 		)
 		(property "Value" "STM-R"
-			(at -1.27 76.43 90)
-			(layer "F.Fab")
+			(at -7.29 73.89 90)
+			(layer "F.SilkS")
 			(effects
 				(font
@@
 		(tags "Through hole socket strip THT 2x30 2.54mm double row")
 		(property "Reference" "J3"
-			(at -1.27 -2.77 90)
+			(at 2.75 0.1 90)
 			(layer "F.SilkS")
 			(effects
@@
 		)
 		(property "Value" "STM-L"
-			(at -1.27 76.43 90)
-			(layer "F.Fab")
+			(at 5.5 73.6 90)
+			(layer "F.SilkS")
 			(effects
 				(font
@@
 			)
 		)
-		(property "Value" "PWR-LED Orange"
-			(at -8.5 0 0)
-			(layer "F.Fab")
+		(property "Value" "PWR"
+			(at -0.25 2 0)
+			(layer "F.SilkS")
 			(effects
 				(font
@@
 		)
 		(property "Value" "MCP1703Ax-330xxMB"
-			(at -3.75 1.25 0)
+			(at -3.75 1.75 0)
 			(layer "F.Fab")
 			(effects
@@
 		(tags "SMA THT Female Jack Vertical")
 		(property "Reference" "J1"
-			(at 0 -4.75 0)
+			(at 2.79 5.71 0)
 			(layer "F.SilkS")
 			(effects
@@
 			)
 		)
-		(property "Value" "TX_SMA"
-			(at 0 5 0)
-			(layer "F.Fab")
+		(property "Value" "TX_ANT"
+			(at 0.04 -6.54 0)
+			(layer "F.SilkS")
 			(effects
 				(font
@@
 		(tags "SMA THT Female Jack Vertical")
 		(property "Reference" "J2"
-			(at 0 -4.75 0)
+			(at -2.71 -5 0)
 			(layer "F.SilkS")
 			(effects
@@
 			)
 		)
-		(property "Value" "RX_SMA"
-			(at 0 5 0)
-			(layer "F.Fab")
+		(property "Value" "RX_ANT"
+			(at -0.21 5.25 0)
+			(layer "F.SilkS")
 			(effects
 				(font
@@
 	(footprint "Symbol:OSHW-Logo2_7.3x6mm_SilkScreen"
 		(layer "F.Cu")
-		(at 174.75 86.5)
+		(at 174.25 86.5)
 		(descr "Open Source Hardware Symbol")
 		(tags "Logo Symbol OSHW")
@@
 		)
 	)
+	(gr_line
+		(start 103.5 78.5)
+		(end 103.5 53)
+		(stroke
+			(width 0.05)
+			(type default)
+		)
+		(layer "Edge.Cuts")
+	)
+	(gr_line
+		(start 180.5 53)
+		(end 180.5 97.25)
+		(stroke
+			(width 0.05)
+			(type default)
+		)
+		(layer "Edge.Cuts")
+	)
+	(gr_line
+		(start 103.5 53)
+		(end 180.5 53)
+		(stroke
+			(width 0.05)
+			(type default)
+		)
+		(layer "Edge.Cuts")
+	)
+	(gr_line
+		(start 103.5 97.25)
+		(end 103.5 78.5)
+		(stroke
+			(width 0.05)
+			(type default)
+		)
+		(layer "Edge.Cuts")
+	)
+	(gr_line
+		(start 180.5 97.25)
+		(end 103.5 97.25)
+		(stroke
+			(width 0.05)
+			(type default)
+		)
+		(layer "Edge.Cuts")
+	)
 	(segment

Commit message: Add files via upload
Parts:
- moved C8 0.12 mm to (147.0, 84.2)
Changed lines of the file:
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@@
 		(tags "resistor")
 		(property "Reference" "R1"
-			(at 0 -1.65 90)
+			(at 2.75 0 90)
 			(layer "F.SilkS")
 			(effects
@@
 		)
 		(property "Value" "100R"
-			(at 0 1.65 90)
+			(at 5.75 0 90)
 			(layer "F.Fab")
 			(effects
@@
 		(tags "capacitor")
 		(property "Reference" "C5"
-			(at 0 -1.68 0)
+			(at 2.75 0 0)
 			(layer "F.SilkS")
 			(effects
@@
 		)
 		(property "Value" "100n"
-			(at 0 1.68 0)
+			(at -3.5 0 0)
 			(layer "F.Fab")
 			(effects
@@
 		(tags "resistor")
 		(property "Reference" "R5"
-			(at 0 -1.65 0)
+			(at -2.8375 0 0)
 			(layer "F.SilkS")
 			(effects
@@
 		)
 		(property "Value" "100R"
-			(at 0 1.65 0)
+			(at 3.6625 0 0)
 			(layer "F.Fab")
 			(effects
@@
 		(tags "capacitor")
 		(property "Reference" "C14"
-			(at 0 -1.68 90)
+			(at -3.5 0 90)
 			(layer "F.SilkS")
 			(effects
@@
 		)
 		(property "Value" "1u"
-			(at 0 1.68 90)
+			(at -3.5 -1.5 90)
 			(layer "F.Fab")
 			(effects
@@
 		(tags "capacitor")
 		(property "Reference" "C11"
-			(at 0 -1.68 0)
+			(at 0 2 0)
 			(layer "F.SilkS")
 			(effects
@@
 		)
 		(property "Value" "33p"
-			(at 0 1.68 0)
+			(at 0 -1.75 0)
 			(layer "F.Fab")
 			(effects
@@
 		(tags "capacitor")
 		(property "Reference" "C2"
-			(at 0 -1.68 0)
+			(at 2.75 0 0)
 			(layer "F.SilkS")
 			(effects
@@
 		)
 		(property "Value" "10n"
-			(at 0 1.68 0)
+			(at -3 0 0)
 			(layer "F.Fab")
 			(effects
@@
 		(tags "capacitor")
 		(property "Reference" "C13"
-			(at 0 -1.68 0)
+			(at 3.3375 0 0)
 			(layer "F.SilkS")
 			(effects
@@
 		)
 		(property "Value" "100n"
-			(at 0 1.68 0)
+			(at -3.6625 0 0)
 			(layer "F.Fab")
 			(effects
@@
 		(tags "resistor")
 		(property "Reference" "R7"
-			(at 0 -1.65 0)
+			(at -2.8375 0 0)
 			(layer "F.SilkS")
 			(effects
@@
 		)
 		(property "Value" "100R"
-			(at 0 1.65 0)
+			(at 3.6625 0 0)
 			(layer "F.Fab")
 			(effects
@@
 		(tags "inductor")
 		(property "Reference" "L1"
-			(at 0 -1.55 90)
+			(at -3 0 90)
 			(layer "F.SilkS")
 			(effects
@@
 		)
 		(property "Value" "82n"
-			(at 0 1.55 90)
+			(at 3.25 0 90)
 			(layer "F.Fab")
 			(effects
@@
 		(tags "capacitor")
 		(property "Reference" "C3"
-			(at 0 -1.68 90)
+			(at -0.25 1.75 90)
 			(layer "F.SilkS")
 			(effects
@@
 		)
 		(property "Value" "10n"
-			(at 0 1.68 90)
+			(at 3.5 0 90)
 			(layer "F.Fab")
 			(effects
@@
 		(tags "capacitor")
 		(property "Reference" "C7"
-			(at 0 -1.68 0)
+			(at 2.75 0 0)
 			(layer "F.SilkS")
 			(effects
@@
 		)
 		(property "Value" "100n"
-			(at 0 1.68 0)
+			(at -3.5 0 0)
 			(layer "F.Fab")
 			(effects
@@
 		(tags "SMD SMT crystal")
 		(property "Reference" "Y1"
-			(at 0 -2.45 0)
+			(at -0.15 -2.6 0)
 			(layer "F.SilkS")
 			(effects
@@
 		)
 		(property "Value" "32MHz"
-			(at 0 2.45 0)
+			(at -0.15 2.65 0)
 			(layer "F.Fab")
 			(effects
@@
 		(tags "LED")
 		(property "Reference" "D1"
-			(at 0 -1.65 0)
+			(at 0 -2 0)
 			(layer "F.SilkS")
 			(effects
@@
 		)
 		(property "Value" "PWR"
-			(at -0.25 2 0)
+			(at 0 2 0)
 			(layer "F.SilkS")
 			(effects
@@
 		(tags "resistor")
 		(property "Reference" "R8"
-			(at 0 -1.65 0)
+			(at 0 -2 0)
 			(layer "F.SilkS")
 			(effects
@@
 		)
 		(property "Value" "100R"
-			(at 0 1.65 0)
+			(at 0 2 0)
 			(layer "F.Fab")
 			(effects
@@
 		(tags "capacitor")
 		(property "Reference" "C4"
-			(at 0 -1.68 90)
+			(at 3.05 0.125 90)
 			(layer "F.SilkS")
 			(effects
@@
 		)
 		(property "Value" "10n"
-			(at 0 1.68 90)
+			(at -2.95 0.125 90)
 			(layer "F.Fab")
 			(effects
@@
 		(tags "resistor")
 		(property "Reference" "R6"
-			(at 0 -1.65 0)
+			(at -2.8375 0 0)
 			(layer "F.SilkS")
 			(effects
@@
 		)
 		(property "Value" "100R"
-			(at 0 1.65 0)
+			(at 3.6625 0 0)
 			(layer "F.Fab")
 			(effects
@@
 		(tags "capacitor")
 		(property "Reference" "C15"
-			(at 0 -1.68 90)
+			(at 3.5 0 90)
 			(layer "F.SilkS")
 			(effects
@@
 		)
 		(property "Value" "1u"
-			(at 0 1.68 90)
+			(at 3.5 1.5 90)
 			(layer "F.Fab")
 			(effects
@@
 		(tags "resistor")
 		(property "Reference" "R2"
-			(at 0 -1.65 90)
+			(at 2.75 0 90)
 			(layer "F.SilkS")
 			(effects
@@
 		)
 		(property "Value" "100R"
-			(at 0 1.65 90)
+			(at 5.75 0 90)
 			(layer "F.Fab")
 			(effects
@@
 		(tags "SOT-89-3")
 		(property "Reference" "U1"
-			(at 3 0 180)
+			(at 3.25 0 180)
 			(layer "F.SilkS")
 			(effects
@@
 		(tags "resistor")
 		(property "Reference" "R4"
-			(at 0 -1.65 0)
+			(at -2.8375 0 0)
 			(layer "F.SilkS")
 			(effects
@@
 		)
 		(property "Value" "100R"
-			(at 0 1.65 0)
+			(at 3.6625 0 0)
 			(layer "F.Fab")
 			(effects
@@
 		(tags "resistor")
 		(property "Reference" "R3"
-			(at 0 -1.65 90)
+			(at 2.75 0 90)
 			(layer "F.SilkS")
 			(effects
@@
 		)
 		(property "Value" "100R"
-			(at 0 1.65 90)
+			(at 5.75 0 90)
 			(layer "F.Fab")
 			(effects
@@
 		(tags "capacitor")
 		(property "Reference" "C6"
-			(at 0 -1.68 90)
+			(at 2.75 0 90)
 			(layer "F.SilkS")
 			(effects
@@
 		)
 		(property "Value" "100n"
-			(at 0 1.68 90)
+			(at 5.75 0 90)
 			(layer "F.Fab")
 			(effects
@@
 		(tags "capacitor")
 		(property "Reference" "C12"
-			(at 0 -1.68 90)
+			(at 3.55 0 90)
 			(layer "F.SilkS")
 			(effects
@@
 		)
 		(property "Value" "27p"
-			(at 0 1.68 90)
+			(at -3.2 0 90)
 			(layer "F.Fab")
 			(effects
@@
 		(tags "capacitor")
 		(property "Reference" "C9"
-			(at 0 -1.68 0)
+			(at 2.75 0 0)
 			(layer "F.SilkS")
 			(effects
@@
 		)
 		(property "Value" "100n"
-			(at 0 1.68 0)
+			(at -3.5 0 0)
 			(layer "F.Fab")
 			(effects
@@
 		(tags "inductor")
 		(property "Reference" "L2"
-			(at 0 -1.55 90)
+			(at -3 0 90)
 			(layer "F.SilkS")
 			(effects
@@
 		)
 		(property "Value" "39n"
-			(at 0 1.55 90)
+			(at 3.25 0 90)
 			(layer "F.Fab")
 			(effects
@@
 		(tags "capacitor")
 		(property "Reference" "C10"
-			(at 0 -1.68 0)
+			(at 3.25 0 0)
 			(layer "F.SilkS")
 			(effects
@@
 		)
 		(property "Value" "100n"
-			(at 0 1.68 0)
+			(at -3.5 0 0)
 			(layer "F.Fab")
 			(effects
@@
 	(footprint "Capacitor_SMD:C_0805_2012Metric"
 		(layer "F.Cu")
-		(at 147.125 84.2 -90)
+		(at 147 84.2 -90)
 		(descr "Capacitor SMD 0805 (2012 Metric), square (rectangular) end terminal, IPC_7351 nominal, (Body size source: IPC-SM-782 page 76, https://www.pcb-3d.com/wordpress/wp-content/uploads/ipc-sm-782a_amendment_1_and_2.pdf, https://docs.google.com/spreadsheets/d/1BsfQQcO9C6DZCsRaXUlFlo91Tg2WpOkGARC1WS5S8t0/edit?usp=sharing), generated with kicad-footprint-generator")
 		(tags "capacitor")
 		(property "Reference" "C8"
-			(at 0 -1.68 90)
+			(at 3.05 0.125 90)
 			(layer "F.SilkS")
 			(effects
@@
 		)
 		(property "Value" "100n"
-			(at 0 1.68 90)
+			(at -3.45 -0.25 90)
 			(layer "F.Fab")
 			(effects
@@
 		(tags "resistor")
 		(property "Reference" "R11"
-			(at 0 -1.65 90)
+			(at 0.15 -1.9375 90)
 			(layer "F.SilkS")
 			(effects
@@
 		)
 		(property "Value" "10K"
-			(at 0 1.65 90)
+			(at 3.4 0.0625 90)
 			(layer "F.Fab")
 			(effects
@@
 		(tags "capacitor")
 		(property "Reference" "C1"
-			(at 0 -1.68 90)
+			(at 2.75 0 90)
 			(layer "F.SilkS")
 			(effects
@@
 		)
 		(property "Value" "10n"
-			(at 0 1.68 90)
+			(at 5.25 0 90)
 			(layer "F.Fab")
 			(effects
